File: Charger.sch (KiCad schematic (older format))
At the start: 12 parts, among them J1 Input, U1 LT1085-5.0

Commit message: actual components added
Parts:
- removed R2: 5, Resistor_SMD:R_0201_0603Metric, symbol Device:R
- added J2: USB-A-S-X-X-SM2, USB:SAMTEC_USB-A-S-X-X-SM2, symbol USB-A-S-X-X-SM2:USB-A-S-X-X-SM2
- C1: value 470u -> 1m
- C2: value 1000u -> 47u
- D1, D2, D3, D4: footprint Diode_THT:D_DO-41_SOD81_P10.16mm_Horizontal -> Diode_1n4005:DIOAD1060W80L410D260
- D5: footprint Diode_SMD:D_SOT-23_ANK -> zener:DIOAD1060W80L410D260
- J1: footprint (none) -> TerminalBlock:TerminalBlock_bornier-2_P5.08mm
- R1: value 100 -> 20
Connections:
- net GND: now also J2.04 (GND)
- net Vout: now reaches C3.1, U1.2 (VO)
- net Vout: now also J2.01 (VCC)
- new net: J2.S1 (SHIELD), J2.S2 (SHIELD)
Changed lines of the file:
@@
 P 5050 3250
 F 0 "C1" H 5228 3296 50  0000 L CNN
-F 1 "470u" H 5228 3205 50  0000 L CNN
+F 1 "1m" H 5228 3205 50  0000 L CNN
 F 2 "Capacitor_SMD:CP_Elec_3x5.3" H 5050 3250 50  0001 C CNN
 F 3 "~" H 5050 3250 50  0001 C CNN
@@
 F 0 "D5" V 5954 3630 50  0000 L CNN
 F 1 "BZX84Cxx" V 6045 3630 50  0000 L CNN
-F 2 "Diode_SMD:D_SOT-23_ANK" H 6000 3375 50  0001 C CNN
+F 2 "zener:DIOAD1060W80L410D260" H 6000 3375 50  0001 C CNN
 F 3 "https://diotec.com/tl_files/diotec/files/pdf/datasheets/bzx84c2v4.pdf" H 6000 3550 50  0001 C CNN
 	1    6000 3550
@@
 P 6000 2550
 F 0 "R1" H 6070 2596 50  0000 L CNN
-F 1 "100" H 6070 2505 50  0000 L CNN
+F 1 "20" H 6070 2505 50  0000 L CNN
 F 2 "Resistor_SMD:R_0201_0603Metric" V 5930 2550 50  0001 C CNN
 F 3 "~" H 6000 2550 50  0001 C CNN
@@
 P 7000 2950
 F 0 "C2" H 7178 2996 50  0000 L CNN
-F 1 "1000u" H 7178 2905 50  0000 L CNN
+F 1 "47u" H 7178 2905 50  0000 L CNN
 F 2 "Capacitor_SMD:CP_Elec_3x5.3" H 7000 2950 50  0001 C CNN
 F 3 "~" H 7000 2950 50  0001 C CNN
 	1    7000 2950
-	1    0    0    -1
-$EndComp
-$Comp
-L Device:R R2
-U 1 1 6031AFD1
-P 10350 3100
-F 0 "R2" H 10420 3146 50  0000 L CNN
-F 1 "5" H 10420 3055 50  0000 L CNN
-F 2 "Resistor_SMD:R_0201_0603Metric" V 10280 3100 50  0001 C CNN
-F 3 "~" H 10350 3100 50  0001 C CNN
-	1    10350 3100
 	1    0    0    -1
 $EndComp
@@
 Wire Wire Line
 	7000 4150 8100 4150
-Wire Wire Line
-	10350 4150 10350 3250
 Connection ~ 7000 4150
 Connection ~ 9650 4150
 Wire Wire Line
-	9650 4150 10350 4150
-Connection ~ 9650 2200
-Wire Wire Line
-	9650 2200 10350 2200
-Wire Wire Line
 	9650 3350 9650 4150
 Wire Wire Line
 	9650 2200 9650 2850
-Wire Wire Line
-	10350 2200 10350 2950
 Wire Wire Line
 	8100 2500 8100 4150
@@
 F 0 "J1" H 2230 3092 50  0000 L CNN
 F 1 "Input" H 2230 3001 50  0000 L CNN
-F 2 "" H 2150 3100 50  0001 C CNN
+F 2 "TerminalBlock:TerminalBlock_bornier-2_P5.08mm" H 2150 3100 50  0001 C CNN
 F 3 "~" H 2150 3100 50  0001 C CNN
 	1    2150 3100
@@
 F 0 "D3" V 4154 2630 50  0000 L CNN
 F 1 "1N4005" V 4245 2630 50  0000 L CNN
-F 2 "Diode_THT:D_DO-41_SOD81_P10.16mm_Horizontal" H 4200 2375 50  0001 C CNN
+F 2 "Diode_1n4005:DIOAD1060W80L410D260" H 4200 2375 50  0001 C CNN
 F 3 "http://www.vishay.com/docs/88503/1n4001.pdf" H 4200 2550 50  0001 C CNN
 	1    4200 2550
@@
 F 0 "D1" V 3054 2630 50  0000 L CNN
 F 1 "1N4005" V 3145 2630 50  0000 L CNN
-F 2 "Diode_THT:D_DO-41_SOD81_P10.16mm_Horizontal" H 3100 2375 50  0001 C CNN
+F 2 "Diode_1n4005:DIOAD1060W80L410D260" H 3100 2375 50  0001 C CNN
 F 3 "http://www.vishay.com/docs/88503/1n4001.pdf" H 3100 2550 50  0001 C CNN
 	1    3100 2550
@@
 F 0 "D2" V 3054 3880 50  0000 L CNN
 F 1 "1N4005" V 3145 3880 50  0000 L CNN
-F 2 "Diode_THT:D_DO-41_SOD81_P10.16mm_Horizontal" H 3100 3625 50  0001 C CNN
+F 2 "Diode_1n4005:DIOAD1060W80L410D260" H 3100 3625 50  0001 C CNN
 F 3 "http://www.vishay.com/docs/88503/1n4001.pdf" H 3100 3800 50  0001 C CNN
 	1    3100 3800
@@
 F 0 "D4" V 4154 3880 50  0000 L CNN
 F 1 "1N4005" V 4245 3880 50  0000 L CNN
-F 2 "Diode_THT:D_DO-41_SOD81_P10.16mm_Horizontal" H 4200 3625 50  0001 C CNN
+F 2 "Diode_1n4005:DIOAD1060W80L410D260" H 4200 3625 50  0001 C CNN
 F 3 "http://www.vishay.com/docs/88503/1n4001.pdf" H 4200 3800 50  0001 C CNN
 	1    4200 3800
 	0    1    1    0
 $EndComp
+$Comp
+L USB-A-S-X-X-SM2:USB-A-S-X-X-SM2 J2
+U 1 1 6032BA44
+P 9500 1450
+F 0 "J2" H 9730 1446 50  0000 L CNN
+F 1 "USB-A-S-X-X-SM2" H 9730 1355 50  0000 L CNN
+F 2 "USB:SAMTEC_USB-A-S-X-X-SM2" H 9500 1450 50  0001 L BNN
+F 3 "" H 9500 1450 50  0001 L BNN
+F 4 "7.8 mm" H 9500 1450 50  0001 L BNN "MAXIMUM_PACKAGE_HEIGHT"
+F 5 "T" H 9500 1450 50  0001 L BNN "PARTREV"
+F 6 "Manufacturer Recommendations" H 9500 1450 50  0001 L BNN "STANDARD"
+F 7 "Samtec" H 9500 1450 50  0001 L BNN "MANUFACTURER"
+	1    9500 1450
+	1    0    0    -1
+$EndComp
+Text GLabel 9650 2200 2    50   Input ~ 0
+Vout
+Text GLabel 9650 4150 2    50   Input ~ 0
+gnd
+Text GLabel 9100 1250 0    50   Input ~ 0
+Vout
+Text GLabel 9100 1550 0    50   Input ~ 0
+gnd
 $EndSCHEMATC

Commit message: footprints repaired
Parts:
- R1: footprint Resistor_SMD:R_0201_0603Metric -> resist_20:EXC-ELSA39
Connections:
- net GND: no longer D1.2 (A), D2.1 (K), J1.2 (Pin_2)
- net Vcc renamed +
- new net -: D1.2 (A), D2.1 (K), J1.2 (Pin_2)
Changed lines of the file:
@@
 F 0 "R1" H 6070 2596 50  0000 L CNN
 F 1 "20" H 6070 2505 50  0000 L CNN
-F 2 "Resistor_SMD:R_0201_0603Metric" V 5930 2550 50  0001 C CNN
+F 2 "resist_20:EXC-ELSA39" V 5930 2550 50  0001 C CNN
 F 3 "~" H 6000 2550 50  0001 C CNN
 	1    6000 2550
@@
 	3100 2200 3100 2400
 Wire Wire Line
-	3100 2700 3100 3200
-Wire Wire Line
 	5050 3000 5050 2200
 Wire Wire Line
@@
 Wire Wire Line
 	8100 4150 9650 4150
-$Comp
-L power:GND #PWR01
-U 1 1 6032C60B
-P 3100 3200
-F 0 "#PWR01" H 3100 2950 50  0001 C CNN
-F 1 "GND" H 3105 3027 50  0000 C CNN
-F 2 "" H 3100 3200 50  0001 C CNN
-F 3 "" H 3100 3200 50  0001 C CNN
-	1    3100 3200
-	0    1    1    0
-$EndComp
-Text GLabel 4200 3200 0    50   Input ~ 0
-Vcc
-Connection ~ 3100 3200
-Wire Wire Line
-	3100 3200 3100 3650
 $Comp
 L pspice:CAP C3
@@
 	1    2150 3100
 	1    0    0    -1
-$EndComp
-Text GLabel 1950 3100 0    50   Input ~ 0
-Vcc
-$Comp
-L power:GND #PWR02
-U 1 1 6031992D
-P 1950 3200
-F 0 "#PWR02" H 1950 2950 50  0001 C CNN
-F 1 "GND" H 1955 3027 50  0000 C CNN
-F 2 "" H 1950 3200 50  0001 C CNN
-F 3 "" H 1950 3200 50  0001 C CNN
-	1    1950 3200
-	1    0    0    -1
-$EndComp
-$Comp
-L Diode:1N4005 D3
-U 1 1 60321173
-P 4200 2550
-F 0 "D3" V 4154 2630 50  0000 L CNN
-F 1 "1N4005" V 4245 2630 50  0000 L CNN
-F 2 "Diode_1n4005:DIOAD1060W80L410D260" H 4200 2375 50  0001 C CNN
-F 3 "http://www.vishay.com/docs/88503/1n4001.pdf" H 4200 2550 50  0001 C CNN
-	1    4200 2550
-	0    1    1    0
-$EndComp
-$Comp
-L Diode:1N4005 D1
-U 1 1 60321C5D
-P 3100 2550
-F 0 "D1" V 3054 2630 50  0000 L CNN
-F 1 "1N4005" V 3145 2630 50  0000 L CNN
-F 2 "Diode_1n4005:DIOAD1060W80L410D260" H 3100 2375 50  0001 C CNN
-F 3 "http://www.vishay.com/docs/88503/1n4001.pdf" H 3100 2550 50  0001 C CNN
-	1    3100 2550
-	0    1    1    0
-$EndComp
-$Comp
-L Diode:1N4005 D2
-U 1 1 603225FE
-P 3100 3800
-F 0 "D2" V 3054 3880 50  0000 L CNN
-F 1 "1N4005" V 3145 3880 50  0000 L CNN
-F 2 "Diode_1n4005:DIOAD1060W80L410D260" H 3100 3625 50  0001 C CNN
-F 3 "http://www.vishay.com/docs/88503/1n4001.pdf" H 3100 3800 50  0001 C CNN
-	1    3100 3800
-	0    1    1    0
-$EndComp
-$Comp
-L Diode:1N4005 D4
-U 1 1 60322E34
-P 4200 3800
-F 0 "D4" V 4154 3880 50  0000 L CNN
-F 1 "1N4005" V 4245 3880 50  0000 L CNN
-F 2 "Diode_1n4005:DIOAD1060W80L410D260" H 4200 3625 50  0001 C CNN
-F 3 "http://www.vishay.com/docs/88503/1n4001.pdf" H 4200 3800 50  0001 C CNN
-	1    4200 3800
-	0    1    1    0
 $EndComp
 $Comp
@@
 Text GLabel 9100 1550 0    50   Input ~ 0
 gnd
+$Comp
+L Diode:1N4005 D1
+U 1 1 603265C3
+P 3100 2550
+F 0 "D1" V 3054 2630 50  0000 L CNN
+F 1 "1N4005" V 3145 2630 50  0000 L CNN
+F 2 "Diode_1n4005:DIOAD1060W80L410D260" H 3100 2375 50  0001 C CNN
+F 3 "http://www.vishay.com/docs/88503/1n4001.pdf" H 3100 2550 50  0001 C CNN
+	1    3100 2550
+	0    1    1    0
+$EndComp
+$Comp
+L Diode:1N4005 D3
+U 1 1 60328034
+P 4200 2550
+F 0 "D3" V 4154 2630 50  0000 L CNN
+F 1 "1N4005" V 4245 2630 50  0000 L CNN
+F 2 "Diode_1n4005:DIOAD1060W80L410D260" H 4200 2375 50  0001 C CNN
+F 3 "http://www.vishay.com/docs/88503/1n4001.pdf" H 4200 2550 50  0001 C CNN
+	1    4200 2550
+	0    1    1    0
+$EndComp
+$Comp
+L Diode:1N4005 D2
+U 1 1 603288BC
+P 3100 3800
+F 0 "D2" V 3054 3880 50  0000 L CNN
+F 1 "1N4005" V 3145 3880 50  0000 L CNN
+F 2 "Diode_1n4005:DIOAD1060W80L410D260" H 3100 3625 50  0001 C CNN
+F 3 "http://www.vishay.com/docs/88503/1n4001.pdf" H 3100 3800 50  0001 C CNN
+	1    3100 3800
+	0    1    1    0
+$EndComp
+$Comp
+L Diode:1N4005 D4
+U 1 1 603291FF
+P 4200 3800
+F 0 "D4" V 4154 3880 50  0000 L CNN
+F 1 "1N4005" V 4245 3880 50  0000 L CNN
+F 2 "Diode_1n4005:DIOAD1060W80L410D260" H 4200 3625 50  0001 C CNN
+F 3 "http://www.vishay.com/docs/88503/1n4001.pdf" H 4200 3800 50  0001 C CNN
+	1    4200 3800
+	0    1    1    0
+$EndComp
+Wire Wire Line
+	3100 2700 3100 3650
+Text GLabel 1950 3200 0    50   Input ~ 10
+-
+Text GLabel 1950 3100 0    50   Input ~ 10
++
+Text GLabel 4200 3200 0    50   Input ~ 10
++
+Text GLabel 3100 3200 0    50   Input ~ 10
+-
 $EndSCHEMATC
