File: Charger.sch (KiCad schematic (older format))
At the start: 12 parts, among them J1 Input, J2 USB-A-S-X-X-SM2, U1 LT1085-5.0

Commit message: usb controller added
Parts:
- removed D1, D2, D3, D4: 1N4005, Diode_1n4005:DIOAD1060W80L410D260, symbol Diode:1N4005
- added D1: D_Bridge_+-AA, symbol Device:D_Bridge_+-AA
- added R2: 100k, symbol Device:R
- added R3: 80.6k, symbol Device:R
- added R4: 16.9k, symbol Device:R
- added U2: TPS2546RTER, RTE0016C, symbol 2021-02-22_11-22-20:TPS2546RTER
Connections:
- net labels added: Vint
- net labels removed: GND
- wire segments 31 -> 39
Other:
- moved on the sheet: C1, C2, C3, J1, R1, U1

Commit message: updates schematics
Parts:
- added T?: Transformer_1P_1S, symbol Device:Transformer_1P_1S
- D1: footprint (none) -> rectifier:SOIC245P670X270-4N
- R1: footprint resist_20:EXC-ELSA39 -> R20:RESC1005X35N
- R2: footprint (none) -> R100k:RESC1005X40N
- R3: footprint (none) -> R806:RESC5025X70N
- R4: footprint (none) -> R169:RESC1608X50N
- U2: footprint RTE0016C -> footprints:TPS2546RTER
Connections:
- net labels added: AC1, AC2
- no-connect marks 0 -> 9
Changed lines of the file:
@@
 F 0 "R1" H 3020 2746 50  0000 L CNN
 F 1 "20" H 3020 2655 50  0000 L CNN
-F 2 "resist_20:EXC-ELSA39" V 2880 2700 50  0001 C CNN
+F 2 "R20:RESC1005X35N" V 2880 2700 50  0001 C CNN
 F 3 "~" H 2950 2700 50  0001 C CNN
 	1    2950 2700
@@
 Text GLabel 9100 1550 0    50   Input ~ 0
 gnd
-Text GLabel 1300 1100 0    50   Input ~ 10
+Text GLabel 3600 1550 2    50   Input ~ 10
 -
-Text GLabel 1300 1000 0    50   Input ~ 10
+Text GLabel 3600 1150 2    50   Input ~ 10
 +
 Text GLabel 850  3150 0    50   Input ~ 10
@@
 F 0 "D1" V 1196 2806 50  0000 R CNN
 F 1 "D_Bridge_+-AA" V 1105 2806 50  0000 R CNN
-F 2 "" H 1150 3150 50  0001 C CNN
+F 2 "rectifier:SOIC245P670X270-4N" H 1150 3150 50  0001 C CNN
 F 3 "~" H 1150 3150 50  0001 C CNN
 	1    1150 3150
@@
 F 0 "U2" H 7950 4136 60  0000 C CNN
 F 1 "TPS2546RTER" H 7950 4030 60  0000 C CNN
-F 2 "RTE0016C" H 7950 2990 60  0001 C CNN
+F 2 "footprints:TPS2546RTER" H 7950 2990 60  0001 C CNN
 F 3 "" H 7950 3050 60  0000 C CNN
 	1    7950 3050
@@
 F 0 "R2" V 6893 2550 50  0000 C CNN
 F 1 "100k" V 6984 2550 50  0000 C CNN
-F 2 "" V 7030 2550 50  0001 C CNN
+F 2 "R100k:RESC1005X40N" V 7030 2550 50  0001 C CNN
 F 3 "~" H 7100 2550 50  0001 C CNN
 	1    7100 2550
@@
 F 0 "R3" H 9070 3846 50  0000 L CNN
 F 1 "80.6k" H 9070 3755 50  0000 L CNN
-F 2 "" V 8930 3800 50  0001 C CNN
+F 2 "R806:RESC5025X70N" V 8930 3800 50  0001 C CNN
 F 3 "~" H 9000 3800 50  0001 C CNN
 	1    9000 3800
@@
 F 0 "R4" H 9420 3846 50  0000 L CNN
 F 1 "16.9k" H 9420 3755 50  0000 L CNN
-F 2 "" V 9280 3800 50  0001 C CNN
+F 2 "R169:RESC1608X50N" V 9280 3800 50  0001 C CNN
 F 3 "~" H 9350 3800 50  0001 C CNN
 	1    9350 3800
@@
 Text GLabel 8650 2350 2    50   Input ~ 0
 Vout
+NoConn ~ 8650 2550
+NoConn ~ 8650 2750
+NoConn ~ 7250 2750
+NoConn ~ 7250 2950
+NoConn ~ 7250 3150
+NoConn ~ 7250 3250
+NoConn ~ 9100 1350
+NoConn ~ 9100 1450
+NoConn ~ 8650 3850
+$Comp
+L Device:Transformer_1P_1S T?
+U 1 1 60353ABB
+P 3200 1350
+F 0 "T?" H 3200 1731 50  0000 C CNN
+F 1 "Transformer_1P_1S" H 3200 1640 50  0000 C CNN
+F 2 "" H 3200 1350 50  0001 C CNN
+F 3 "~" H 3200 1350 50  0001 C CNN
+	1    3200 1350
+	1    0    0    -1
+$EndComp
+Text GLabel 1300 1000 0    50   Input ~ 0
+AC1
+Text GLabel 1300 1100 0    50   Input ~ 0
+AC2
+Text GLabel 2800 1150 0    50   Input ~ 0
+AC1
+Text GLabel 2800 1550 0    50   Input ~ 0
+AC2
 $EndSCHEMATC

Commit message: Update Charger.sch
Parts:
- C1: value 1m -> 4.7m; footprint Capacitor_SMD:CP_Elec_3x5.3 -> Capacitor_SMD:CP_Elec_6.3x9.9
- T1: renamed from T?; value Transformer_1P_1S -> Transformer_12P_1S; footprint (none) -> Transformer_SMD:Transformer_Coilcraft_CST2010
Changed lines of the file:
@@
 P 2000 3400
 F 0 "C1" H 2178 3446 50  0000 L CNN
-F 1 "1m" H 2178 3355 50  0000 L CNN
-F 2 "Capacitor_SMD:CP_Elec_3x5.3" H 2000 3400 50  0001 C CNN
+F 1 "4.7m" H 2178 3355 50  0000 L CNN
+F 2 "Capacitor_SMD:CP_Elec_6.3x9.9" H 2000 3400 50  0001 C CNN
 F 3 "~" H 2000 3400 50  0001 C CNN
 	1    2000 3400
@@
 NoConn ~ 8650 3850
 $Comp
-L Device:Transformer_1P_1S T?
+L Device:Transformer_1P_1S T1
 U 1 1 60353ABB
 P 3200 1350
-F 0 "T?" H 3200 1731 50  0000 C CNN
-F 1 "Transformer_1P_1S" H 3200 1640 50  0000 C CNN
-F 2 "" H 3200 1350 50  0001 C CNN
+F 0 "T1" H 3200 1731 50  0000 C CNN
+F 1 "Transformer_12P_1S" H 3200 1640 50  0000 C CNN
+F 2 "Transformer_SMD:Transformer_Coilcraft_CST2010" H 3200 1350 50  0001 C CNN
 F 3 "~" H 3200 1350 50  0001 C CNN
 	1    3200 1350

Commit message: Update Charger.sch
Parts:
- T1: value Transformer_12P_1S -> Transformer_1P_1S; footprint Transformer_SMD:Transformer_Coilcraft_CST2010 -> Transformer_THT:Transformer_Breve_TEZ-47x57
Changed lines of the file:
@@
 P 3200 1350
 F 0 "T1" H 3200 1731 50  0000 C CNN
-F 1 "Transformer_12P_1S" H 3200 1640 50  0000 C CNN
-F 2 "Transformer_SMD:Transformer_Coilcraft_CST2010" H 3200 1350 50  0001 C CNN
+F 1 "Transformer_1P_1S" H 3200 1640 50  0000 C CNN
+F 2 "Transformer_THT:Transformer_Breve_TEZ-47x57" H 3200 1350 50  0001 C CNN
 F 3 "~" H 3200 1350 50  0001 C CNN
 	1    3200 1350

Commit message: minor updates
Parts:
- removed C2: 47u, Capacitor_SMD:CP_Elec_3x5.3, symbol pspice:CAP
- removed D5: BZX84Cxx, zener:DIOAD1060W80L410D260, symbol Diode:BZX84Cxx
- removed R1: 20, R20:RESC1005X35N, symbol Device:R
- removed T1: Transformer_1P_1S, Transformer_THT:Transformer_Breve_TEZ-47x57, symbol Device:Transformer_1P_1S
- added TR1: TEZ6.0-D-1, Transformer_THT:Transformer_Breve_TEZ-38x45, symbol Transformer:TEZ6.0-D-1
Connections:
- wire segments 39 -> 27
Other:
- moved on the sheet: C1, D1
Changed lines of the file:
@@
 L pspice:CAP C1
 U 1 1 60316869
-P 2000 3400
-F 0 "C1" H 2178 3446 50  0000 L CNN
-F 1 "4.7m" H 2178 3355 50  0000 L CNN
-F 2 "Capacitor_SMD:CP_Elec_6.3x9.9" H 2000 3400 50  0001 C CNN
-F 3 "~" H 2000 3400 50  0001 C CNN
-	1    2000 3400
-	1    0    0    -1
-$EndComp
-$Comp
-L Diode:BZX84Cxx D5
-U 1 1 603170B0
-P 2950 3700
-F 0 "D5" V 2904 3780 50  0000 L CNN
-F 1 "BZX84Cxx" V 2995 3780 50  0000 L CNN
-F 2 "zener:DIOAD1060W80L410D260" H 2950 3525 50  0001 C CNN
-F 3 "https://diotec.com/tl_files/diotec/files/pdf/datasheets/bzx84c2v4.pdf" H 2950 3700 50  0001 C CNN
-	1    2950 3700
-	0    1    1    0
-$EndComp
-$Comp
-L Device:R R1
-U 1 1 60317AB7
-P 2950 2700
-F 0 "R1" H 3020 2746 50  0000 L CNN
-F 1 "20" H 3020 2655 50  0000 L CNN
-F 2 "R20:RESC1005X35N" V 2880 2700 50  0001 C CNN
-F 3 "~" H 2950 2700 50  0001 C CNN
-	1    2950 2700
-	1    0    0    -1
-$EndComp
-$Comp
-L pspice:CAP C2
-U 1 1 60318512
-P 3950 3100
-F 0 "C2" H 4128 3146 50  0000 L CNN
-F 1 "47u" H 4128 3055 50  0000 L CNN
-F 2 "Capacitor_SMD:CP_Elec_3x5.3" H 3950 3100 50  0001 C CNN
-F 3 "~" H 3950 3100 50  0001 C CNN
-	1    3950 3100
+P 4650 3400
+F 0 "C1" H 4828 3446 50  0000 L CNN
+F 1 "4.7m" H 4828 3355 50  0000 L CNN
+F 2 "Capacitor_SMD:CP_Elec_6.3x9.9" H 4650 3400 50  0001 C CNN
+F 3 "~" H 4650 3400 50  0001 C CNN
+	1    4650 3400
 	1    0    0    -1
 $EndComp
@@
 $EndComp
 Wire Wire Line
-	2000 3150 2000 2350
-Wire Wire Line
-	2000 3650 2000 4300
-Wire Wire Line
-	2000 4300 1150 4300
-Wire Wire Line
-	2950 4300 2950 3850
-Wire Wire Line
-	2950 3550 2950 3150
-Wire Wire Line
-	2950 2550 2950 2350
-Wire Wire Line
-	2950 2350 2000 2350
-Connection ~ 2000 2350
-Wire Wire Line
-	2950 3150 3450 3150
-Wire Wire Line
-	3450 3150 3450 2350
-Wire Wire Line
-	3450 2350 3950 2350
-Wire Wire Line
-	3950 2350 3950 2850
-Connection ~ 2950 3150
-Wire Wire Line
-	2950 3150 2950 2850
-Wire Wire Line
-	3950 3350 3950 4300
-Wire Wire Line
-	3950 4300 2950 4300
-Connection ~ 2950 4300
-Wire Wire Line
-	2000 4300 2950 4300
-Connection ~ 2000 4300
-Wire Wire Line
-	3950 2350 4750 2350
-Connection ~ 3950 2350
-Wire Wire Line
-	3950 4300 5050 4300
-Connection ~ 3950 4300
+	4650 3150 4650 2350
+Wire Wire Line
+	4650 3650 4650 4300
+Wire Wire Line
+	4650 4300 3800 4300
 Wire Wire Line
 	6600 3500 6600 4300
 Wire Wire Line
 	6600 2350 6600 3000
-Wire Wire Line
-	5050 2650 5050 4300
-Connection ~ 5050 4300
 Wire Wire Line
 	5050 4300 6600 4300
@@
 Text GLabel 9100 1550 0    50   Input ~ 0
 gnd
-Text GLabel 3600 1550 2    50   Input ~ 10
+Text GLabel 4850 1500 2    50   Input ~ 10
 -
-Text GLabel 3600 1150 2    50   Input ~ 10
+Text GLabel 4850 1100 2    50   Input ~ 10
 +
-Text GLabel 850  3150 0    50   Input ~ 10
+Text GLabel 3500 3150 0    50   Input ~ 10
 -
 $Comp
 L Device:D_Bridge_+-AA D1
 U 1 1 603431A1
-P 1150 3150
-F 0 "D1" V 1196 2806 50  0000 R CNN
-F 1 "D_Bridge_+-AA" V 1105 2806 50  0000 R CNN
-F 2 "rectifier:SOIC245P670X270-4N" H 1150 3150 50  0001 C CNN
-F 3 "~" H 1150 3150 50  0001 C CNN
-	1    1150 3150
+P 3800 3150
+F 0 "D1" V 3846 2806 50  0000 R CNN
+F 1 "D_Bridge_+-AA" V 3755 2806 50  0000 R CNN
+F 2 "rectifier:SOIC245P670X270-4N" H 3800 3150 50  0001 C CNN
+F 3 "~" H 3800 3150 50  0001 C CNN
+	1    3800 3150
 	0    -1   -1   0
 $EndComp
 Wire Wire Line
-	1150 3450 1150 4300
-Wire Wire Line
-	1150 2850 1150 2350
-Wire Wire Line
-	1150 2350 2000 2350
-Text GLabel 1450 3150 3    50   Input ~ 0
+	3800 3450 3800 4300
+Wire Wire Line
+	3800 2850 3800 2350
+Wire Wire Line
+	3800 2350 4650 2350
+Text GLabel 4100 3150 3    50   Input ~ 0
 +
 $Comp
@@
 NoConn ~ 9100 1450
 NoConn ~ 8650 3850
-$Comp
-L Device:Transformer_1P_1S T1
-U 1 1 60353ABB
-P 3200 1350
-F 0 "T1" H 3200 1731 50  0000 C CNN
-F 1 "Transformer_1P_1S" H 3200 1640 50  0000 C CNN
-F 2 "Transformer_THT:Transformer_Breve_TEZ-47x57" H 3200 1350 50  0001 C CNN
-F 3 "~" H 3200 1350 50  0001 C CNN
-	1    3200 1350
-	1    0    0    -1
-$EndComp
 Text GLabel 1300 1000 0    50   Input ~ 0
 AC1
 Text GLabel 1300 1100 0    50   Input ~ 0
 AC2
-Text GLabel 2800 1150 0    50   Input ~ 0
+Text GLabel 4450 1100 0    50   Input ~ 0
 AC1
-Text GLabel 2800 1550 0    50   Input ~ 0
+Text GLabel 4450 1500 0    50   Input ~ 0
 AC2
+$Comp
+L Transformer:TEZ6.0-D-1 TR1
+U 1 1 60359C75
+P 4650 1300
+F 0 "TR1" H 4650 1725 50  0000 C CNN
+F 1 "TEZ6.0-D-1" H 4650 1634 50  0000 C CNN
+F 2 "Transformer_THT:Transformer_Breve_TEZ-38x45" H 4650 950 50  0001 C CIN
+F 3 "http://www.breve.pl/pdf/ANG/TEZ_ang.pdf" H 4650 1300 50  0001 C CNN
+	1    4650 1300
+	1    0    0    -1
+$EndComp
+Wire Wire Line
+	5050 2650 5050 4300
+Wire Wire Line
+	4650 2350 4750 2350
+Connection ~ 4650 2350
+Wire Wire Line
+	4650 4300 5050 4300
+Connection ~ 4650 4300
+Connection ~ 5050 4300
 $EndSCHEMATC

Commit message: just pcb update
Parts:
- U2: value TPS2546RTER -> TPS2546; Spice_Lib_File (none) -> C:\\Users\\bhoop\\Downloads\\slvm796a\\SLVM796\\TPS2546_PSP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; Spice_Model (none) -> TPS2546_TRANS; Spice_Netlist_Enabled (none) -> Y; Spice_Primitive (none) -> X
Connections:
- net DM: now reaches J2.02 (D-)
- net DM: now also U2.11 (DM_IN)
- net DP: now reaches J2.03 (D+)
- net DP: now also U2.10 (DP_IN)
- no-connect marks 9 -> 5
Other:
- moved on the sheet: TR1
Changed lines of the file:
@@
 Text GLabel 9100 1550 0    50   Input ~ 0
 gnd
-Text GLabel 4850 1500 2    50   Input ~ 10
+Text GLabel 7000 1350 2    50   Input ~ 10
 -
-Text GLabel 4850 1100 2    50   Input ~ 10
+Text GLabel 7000 950  2    50   Input ~ 10
 +
 Text GLabel 3500 3150 0    50   Input ~ 10
@@
 Text GLabel 4100 3150 3    50   Input ~ 0
 +
-$Comp
-L 2021-02-22_11-22-20:TPS2546RTER U2
-U 1 1 6034FCE9
-P 7950 3050
-F 0 "U2" H 7950 4136 60  0000 C CNN
-F 1 "TPS2546RTER" H 7950 4030 60  0000 C CNN
-F 2 "footprints:TPS2546RTER" H 7950 2990 60  0001 C CNN
-F 3 "" H 7950 3050 60  0000 C CNN
-	1    7950 3050
-	1    0    0    -1
-$EndComp
 Connection ~ 6600 2350
 Text GLabel 6600 2350 1    50   Input ~ 0
@@
 Text GLabel 8650 2350 2    50   Input ~ 0
 Vout
-NoConn ~ 8650 2550
-NoConn ~ 8650 2750
 NoConn ~ 7250 2750
 NoConn ~ 7250 2950
 NoConn ~ 7250 3150
 NoConn ~ 7250 3250
-NoConn ~ 9100 1350
-NoConn ~ 9100 1450
 NoConn ~ 8650 3850
 Text GLabel 1300 1000 0    50   Input ~ 0
@@
 Text GLabel 1300 1100 0    50   Input ~ 0
 AC2
-Text GLabel 4450 1100 0    50   Input ~ 0
+Text GLabel 6600 950  0    50   Input ~ 0
 AC1
-Text GLabel 4450 1500 0    50   Input ~ 0
+Text GLabel 6600 1350 0    50   Input ~ 0
 AC2
 $Comp
 L Transformer:TEZ6.0-D-1 TR1
 U 1 1 60359C75
-P 4650 1300
-F 0 "TR1" H 4650 1725 50  0000 C CNN
-F 1 "TEZ6.0-D-1" H 4650 1634 50  0000 C CNN
-F 2 "Transformer_THT:Transformer_Breve_TEZ-38x45" H 4650 950 50  0001 C CIN
-F 3 "http://www.breve.pl/pdf/ANG/TEZ_ang.pdf" H 4650 1300 50  0001 C CNN
-	1    4650 1300
+P 6800 1150
+F 0 "TR1" H 6800 1575 50  0000 C CNN
+F 1 "TEZ6.0-D-1" H 6800 1484 50  0000 C CNN
+F 2 "Transformer_THT:Transformer_Breve_TEZ-38x45" H 6800 800 50  0001 C CIN
+F 3 "http://www.breve.pl/pdf/ANG/TEZ_ang.pdf" H 6800 1150 50  0001 C CNN
+	1    6800 1150
 	1    0    0    -1
 $EndComp
@@
 Connection ~ 4650 4300
 Connection ~ 5050 4300
+$Comp
+L 2021-02-22_11-22-20:TPS2546RTER U2
+U 1 1 6034FCE9
+P 7950 3050
+F 0 "U2" H 7950 4136 60  0000 C CNN
+F 1 "TPS2546" H 7950 4030 60  0000 C CNN
+F 2 "footprints:TPS2546RTER" H 7950 2990 60  0001 C CNN
+F 3 "" H 7950 3050 60  0000 C CNN
+F 4 "X" H 7950 3050 50  0001 C CNN "Spice_Primitive"
+F 5 "TPS2546_TRANS" H 7950 3050 50  0001 C CNN "Spice_Model"
+F 6 "Y" H 7950 3050 50  0001 C CNN "Spice_Netlist_Enabled"
+F 7 "C:\\Users\\bhoop\\Downloads\\slvm796a\\SLVM796\\TPS2546_PSPICE_TRANS\\TPS2546_TRANS.LIB" H 7950 3050 50  0001 C CNN "Spice_Lib_File"
+	1    7950 3050
+	1    0    0    -1
+$EndComp
+Text GLabel 9100 1350 0    50   Input ~ 0
+DM
+Text GLabel 9100 1450 0    50   Input ~ 0
+DP
+Text GLabel 8650 2550 2    50   Input ~ 0
+DM
+Text GLabel 8650 2750 2    50   Input ~ 0
+DP
 $EndSCHEMATC

Commit message: newer schematics
Parts:
- removed C1: 4.7m, Capacitor_SMD:CP_Elec_6.3x9.9, symbol pspice:CAP
- added C? (x2): CAP, symbol pspice:CAP
- added J3: USB-A-S-X-X-SM2, SAMTEC_USB-A-S-X-X-SM2, symbol USB-A-S-X-X-SM2:USB-A-S-X-X-SM2
- added R1: 100k, symbol Device:R
- added R5: 80.6k, symbol Device:R
- added R6: 16.9k, symbol Device:R
- added R? (x4): R, symbol Device:R
- added U3: LT3798MPMSETRPBF, MSOP-16_MSE, symbol LT3798MPMSETRPBF:LT3798MPMSETRPBF
- added U4: TPS2546RTER, RTE0016C, symbol 2021-02-22_11-22-20:TPS2546RTER
Connections:
- net Vint is gone; now on net Stat1: C3.1, R2.2, U1.2 (VO), U2.1 (IN), U2.5 (EN), U2.7 (CLT2), U2.8 (CLT3)
- net +: no longer D1.4 (~~)
- net -: no longer D1.3 (~~)
- net DM: no longer U2.11 (DM_IN)
- net DP: no longer U2.10 (DP_IN)
- net Vout: no longer U2.12 (OUT)
- net gnd: now also C?.2, J3.04 (GND), R5.2, R6.2, R?.2, R?.2, U3.17 (GND), U4.14 (GND), U4.6 (CLT1); no longer D1.2 (-)
- net at U1.3 (VI): no longer D1.1 (+)
- net Stat1: now reaches U2.9 (STATUS_N)
- net Stat1: now also R1.2, U4.1 (IN), U4.5 (EN), U4.7 (CLT2), U4.8 (CLT3), U4.9 (STATUS_N)
- new net: R5.1, U4.15 (ILIM_LO)
- new net: R6.1, U4.16 (ILIM_HI)
- new net: R1.1, U4.4 (ILIM_SEL)
- new net: J3.S1 (SHIELD), J3.S2 (SHIELD)
- new net: R?.1, R?.1, U3.1 (CTRL1), U3.2 (CTRL2), U3.4 (VREF)
- new net: R?.1, R?.2, U3.3 (CTRL3)
- new net: R?.1, R?.2, U3.5 (OVP)
- new net: C?.1, U3.6 (VC)
- new net: C?.2, U3.7 (COMP+)
- new net DM1: U2.11 (DM_IN)
- new net DM2: J3.02 (D-), U4.11 (DM_IN)
- new net DP1: U2.10 (DP_IN)
- new net DP2: J3.03 (D+), U4.10 (DP_IN)
- new net Vout1: U2.12 (OUT)
- new net Vout2: J3.01 (VCC), U4.12 (OUT)
- no-connect marks 5 -> 8
Other:
- moved on the sheet: D1, J1, U1

Commit message: SMP connections done
stat inputs of 2546 corrected
smp circuit connections done
diode, mosfet models remaining
internal resistance of capacitance remaining
transformer remaining
Parts:
- added C?: C, symbol Device:C
- added C?: 4.7p, symbol Device:C
- added C?: 22p, symbol Device:C
- added C?: 4.7m, symbol Device:C
- added C?: 10u, symbol Device:C
- added C?: 470u, symbol Device:C
- added D?: DIODE, symbol pspice:DIODE
- added D?: D_Zener, symbol Device:D_Zener
- added D? (x3): D, symbol Device:D
- added L? (x3): L, symbol Device:L
- added M?: MNMOS, symbol pspice:MNMOS
- added R?: 90k, symbol Device:R
- added R?: 10k, symbol Device:R
- added R?: 0.05, symbol Device:R
- added R? (x2): 1meg, symbol Device:R
- added R?: 200k, symbol Device:R
- added R?: 95.3k, symbol Device:R
- added R?: 20, symbol Device:R
- C?: value CAP -> 4.7u
- C?: value CAP -> 0.1u
- J2, J3: symbol USB-A-S-X-X-SM2:USB-A-S-X-X-SM2 -> Charger-rescue:USB-A-S-X-X-SM2-USB-A-S-X-X-SM2
- R? (x2): value R -> 40.2k
- R?: value R -> 54k
- R?: value R -> 90.9k
- U2, U4: symbol 2021-02-22_11-22-20:TPS2546RTER -> Charger-rescue:TPS2546RTER-2021-02-22_11-22-20
- U3: symbol LT3798MPMSETRPBF:LT3798MPMSETRPBF -> Charger-rescue:LT3798MPMSETRPBF-LT3798MPMSETRPBF
Connections:
- net Stat1: no longer C3.1, R1.2, R2.2, U1.2 (VO), U2.1 (IN), U2.5 (EN), U2.7 (CLT2), U2.8 (CLT3), U4.1 (IN), U4.5 (EN), U4.7 (CLT2), U4.8 (CLT3), U4.9 (STATUS_N)
- net gnd: now also D1.2 (-), C?.2, C?.2, C?.2, C?.2, C?.2, L?.2, L?.2, R?.2, R?.2, R?.2
- net at U1.3 (VI): now also C?.1, D?.1 (K)
- net at D1.1 (+): now also C?.1, D?.2 (A), L?.1, R?.1, R?.1
- net at U3.10 (DCM): now also C?.2
- net VinL: now reaches U3.11 (VIN)
- net VinL: now also C?.1, D?.1 (K), D?.1 (K), R?.1
- net en: now reaches U3.12 (EN/UVLO)
- net en: now also R?.1, R?.2
- net at U3.13 (INTVCC): now also C?.1
- net at U3.14 (GATE): now also M?.2 (G)
- net at U3.15 (SENSE): now also M?.3 (S), M?.4 (B), R?.1
- net Vin_sense: now reaches U3.16 (VIN_SENSE)
- net Vin_sense: now also R?.2
- net at U3.9 (FB): now also C?.1, R?.1, R?.1
- new net: D?.1 (K), L?.2, M?.1 (D)
- new net: D?.1 (K), D?.2 (A)
- new net: D?.2 (A), R?.2
- new net: D?.2 (A), R?.1
- new net: D?.2 (A), L?.1
- new net Stat2: U4.9 (STATUS_N)
- new net Vint: C3.1, R1.2, R2.2, U1.2 (VO), U2.1 (IN), U2.5 (EN), U2.7 (CLT2), U2.8 (CLT3), U4.1 (IN), U4.5 (EN), U4.7 (CLT2), U4.8 (CLT3)
- new net dcm: C?.1, L?.1, R?.2, R?.2
Other:
- moved on the sheet: C?, D1, R?, U3
