File: Charger.kicad_pcb (KiCad board)
At the start: 2 copper layers, 11 parts, among them U1 LT1085-5.0

Commit message: Update Charger.kicad_pcb
Parts:
- turned C3 to 180 degrees
- turned R2 to 180 degrees

Commit message: actual components added
Parts:
- removed R2: 5, Resistor_SMD:R_0201_0603Metric
- added J1: Input, TerminalBlock:TerminalBlock_bornier-2_P5.08mm, F.Cu at (563.7, 984.9)
- added J2: USB-A-S-X-X-SM2, USB:SAMTEC_USB-A-S-X-X-SM2, F.Cu at (551.2, 978.3)
- C1: value 470u -> 1m
- C2: value 1000u -> 47u
- D1, D2, D3, D4: value 1N914 -> 1N4005; footprint Diode_SMD:D_0201_0603Metric -> Diode_1n4005:DIOAD1060W80L410D260
- D5: footprint Diode_SMD:D_SOT-23_ANK -> zener:DIOAD1060W80L410D260
- R1: value 100 -> 20
- moved D1 405.7 mm to (548.6, 1014.7)
- moved R1 391.2 mm to (531.6, 999.0)
- moved C2 381.9 mm to (561.3, 991.9), turned to 0 degrees
- moved D2 375.0 mm to (548.8, 991.2)
- moved D4 374.8 mm to (551.1, 995.2)
- moved U1 371.0 mm to (523.2, 979.2)
- moved C3 368.2 mm to (575.4, 982.8), turned to 0 degrees
- moved D3 359.2 mm to (567.4, 974.3)
- moved D5 359.1 mm to (567.4, 978.4)
- moved C1 353.6 mm to (577.6, 974.7)
Connections:
- net Net-(C3-Pad1) renamed Vout
- C1 pad 2: GND -> gnd
- C2 pad 2: GND -> gnd
- C3 pad 2: GND -> gnd
- U1 pad 1: GND -> gnd

Commit message: footprints repaired
Parts:
- R1: footprint Resistor_SMD:R_0201_0603Metric -> resist_20:EXC-ELSA39
- moved J1 147.2 mm to (433.1, 1052.8), turned to 90 degrees
- moved C1 145.3 mm to (455.9, 1054.1), turned to 270 degrees
- moved D3 136.4 mm to (450.9, 1045.2), turned to 90 degrees
- moved D5 136.1 mm to (459.7, 1061.7), turned to 90 degrees
- moved C3 133.3 mm to (468.9, 1063.0), turned to 180 degrees
- moved D2 126.3 mm to (443.2, 1060.5), turned to 270 degrees
- moved D4 119.6 mm to (450.9, 1060.5), turned to 270 degrees
- moved C2 110.6 mm to (478.8, 1065.5)
- moved D1 109.7 mm to (443.2, 1045.2), turned to 90 degrees
- moved J2 96.7 mm to (483.9, 1047.8), turned to 90 degrees
- moved U1 92.0 mm to (470.1, 1054.3)
- moved R1 86.1 mm to (459.7, 1046.5), turned to 270 degrees
Connections:
- J1 pad 1: Vcc -> +
- J1 pad 2: gnd -> -

Commit message: Update Charger.kicad_pcb
Parts:
- moved C2 24.3 mm to (462.3, 1047.8), turned to 90 degrees
- moved C1 8.98 mm to (457.2, 1063.0)
- moved J2 3.81 mm to (483.9, 1051.6)
- moved R1 2.84 mm to (457.2, 1047.8)
- moved D5 2.84 mm to (462.3, 1060.5), turned to 270 degrees
- moved J1 2.54 mm to (433.1, 1050.3), turned to 270 degrees
- moved U1 1.08 mm to (471.2, 1054.1)
- turned D1 to 270 degrees
- turned D3 to 270 degrees
Routing:
- net Net-(C1-Pad1): track 0.00 -> 38.3 mm
- net Net-(C2-Pad1): track 0.00 -> 30.9 mm
- net +: track 0.00 -> 28.8 mm
- net Vout: track 0.00 -> 21.2 mm
- net Net-(J2-PadS1): track 0.00 -> 19.1 mm
- net -: track 0.00 -> 14.9 mm
- added copper zone on B.Cu, net (none)
- added copper zone on F.Cu, net gnd
Other:
- board outline added: 67.3 x 30.6 mm
- board text added: "1N4005"
- board text added: "20 ohm"
- board text added: "BZX85C10"
- board text added: "LT1085-5.0"
- board text added: "USB"
- board text added: "input"
