File: Charger.kicad_pcb (KiCad board)
At the start: 2 copper layers, 67.3 x 30.6 mm, 12 parts, among them J1 Input, J2 USB-A-S-X-X-SM2, U1 LT1085-5.0

Commit message: updates schematics
Parts:
- removed D2, D3, D4: 1N4005, Diode_1n4005:DIOAD1060W80L410D260
- added R2: 100k, R100k:RESC1005X40N, F.Cu at (474.2, 1073.8)
- added R3: 80.6k, R806:RESC5025X70N, F.Cu at (454.6, 1068.6)
- added R4: 16.9k, R169:RESC1608X50N, F.Cu at (461.3, 1077.2)
- added T1: Transformer_12P_1S, Transformer_SMD:Transformer_Coilcraft_CST2010, F.Cu at (448.0, 1057.9)
- added U2: TPS2546RTER, footprints:TPS2546RTER, F.Cu at (482.8, 1068.5)
- C1: value 1m -> 4.7m; footprint Capacitor_SMD:CP_Elec_3x5.3 -> Capacitor_SMD:CP_Elec_6.3x9.9
- D1: value 1N4005 -> D_Bridge_+-AA; footprint Diode_1n4005:DIOAD1060W80L410D260 -> rectifier:SOIC245P670X270-4N
- R1: footprint resist_20:EXC-ELSA39 -> R20:RESC1005X35N
- moved D1 40.6 mm to (475.8, 1069.5), turned to 0 degrees
- moved R1 31.8 mm to (464.8, 1078.6), turned to 0 degrees
- moved C2 25.8 mm to (462.6, 1073.5), turned to 0 degrees
- moved J1 25.7 mm to (440.3, 1075.0), turned to 0 degrees
- moved D5 20.0 mm to (443.9, 1068.4), turned to 0 degrees
- moved U1 12.9 mm to (464.8, 1065.3)
- moved C1 12.6 mm to (453.9, 1075.2), turned to 0 degrees
- moved C3 12.1 mm to (469.3, 1075.1), turned to 0 degrees
- moved J2 5.56 mm to (479.8, 1055.4), turned to 0 degrees
Connections:
- C3 pad 1: Vout -> Vint
- D1 pad 2: - -> gnd
- J1 pad 1: + -> AC1
- J1 pad 2: - -> AC2
- U1 pad 2: Vout -> Vint
Routing:
- net Net-(C1-Pad1): track 38.3 -> 0.00 mm
- net Net-(C2-Pad1): track 30.9 -> 0.00 mm
- net +: track 28.8 -> 0.00 mm
- net Vout: track 21.2 -> 0.00 mm
- net Net-(J2-PadS1): track 19.1 -> 0.00 mm
- net -: track 14.9 -> 0.00 mm
- removed copper zone on B.Cu, net (none)
- removed copper zone on F.Cu, net gnd
Other:
- board outline removed
- board text removed: "1N4005"
- board text removed: "20 ohm"
- board text removed: "BZX85C10"
- board text removed: "LT1085-5.0"
- board text removed: "USB"
- board text removed: "input"

Commit message: just pcb update
Parts:
- removed C2: 47u, Capacitor_SMD:CP_Elec_3x5.3
- removed D5: BZX84Cxx, zener:DIOAD1060W80L410D260
- removed R1: 20, R20:RESC1005X35N
- removed T1: Transformer_12P_1S, Transformer_SMD:Transformer_Coilcraft_CST2010
- added TR1: TEZ6.0-D-1, Transformer_THT:Transformer_Breve_TEZ-38x45, F.Cu at (106.0, 68.1)
- U2: value TPS2546RTER -> TPS2546
- moved C1 1062.7 mm to (144.0, 58.7)
- moved D1 1051.4 mm to (142.9, 72.1), turned to 90 degrees
- moved C3 1045.1 mm to (142.9, 82.3)
- moved U1 1041.8 mm to (156.5, 70.1)
- moved R4 1037.4 mm to (144.7, 89.3)
- moved J1 1033.3 mm to (155.6, 81.7)
- moved U2 1032.4 mm to (141.7, 94.1)
- moved R2 1029.7 mm to (144.2, 98.4)
- moved R3 1014.4 mm to (143.6, 103.0)
- moved J2 1012.4 mm to (154.6, 96.6), turned to 90 degrees
Connections:
- J2 pad 02: Net-(J2-Pad02) -> DM
- J2 pad 03: Net-(J2-Pad03) -> DP
- U1 pad 3: Net-(C2-Pad1) -> Net-(C1-Pad1)
- U2 pad 10: Net-(U2-Pad10) -> DP
- U2 pad 11: Net-(U2-Pad11) -> DM
Routing:
- net Net-(R4-Pad1): track 0.00 -> 4.64 mm
Other:
- board outline added: 72.6 x 55.8 mm

Commit message: t
Parts:
- added C2: 4.7u, cap4:CAPC2012X140N, F.Cu at (109.4, 111.2)
- added C4: 0.1u, Capacitor_THT:CP_Radial_D4.0mm_P1.50mm, F.Cu at (150.2, 96.3)
- added C5: 10u, Capacitor_THT:CP_Radial_D4.0mm_P1.50mm, F.Cu at (138.6, 112.4)
- added C6: 4.7u, cap4:CAPC2012X140N, F.Cu at (132.9, 93.2)
- added C7: 4.7p, Capacitor_THT:CP_Radial_D4.0mm_P1.50mm, F.Cu at (133.0, 112.4)
- added C8: 470u, Capacitor_THT:CP_Radial_D8.0mm_P3.80mm, F.Cu at (134.0, 100.5)
- added C9: 22p, Capacitor_THT:CP_Radial_D4.0mm_P1.50mm, F.Cu at (142.7, 102.8)
- added D2: 1N4007, 1N4007:DIOAD1060W80L520D270, F.Cu at (130.8, 78.1)
- added D3: 1N4148WS, 1N4148WS:SODFL2512X100N, F.Cu at (159.6, 77.4)
- added D4: DFLZ33, 1N4148WS:SODFL2512X100N, F.Cu at (110.0, 116.0)
- added D5: GSD2004W-V, 1N4148WS:SODFL2512X100N, F.Cu at (140.5, 77.4)
- added D6: MBRS360, 1N4148WS:SODFL2512X100N, F.Cu at (115.6, 116.0)
- added J3: USB-A-S-X-X-SM2, USB:SAMTEC_USB-A-S-X-X-SM2, F.Cu at (97.9, 106.5)
- added Q1: BSC42DN25NS3, MOSFET:SOT230P700X180-4N, F.Cu at (152.0, 80.1)
- added R1: 100k, R100k:RESC1005X40N, F.Cu at (161.3, 82.9)
- added R10: 54k, R806:RESC5025X70N, F.Cu at (134.6, 107.4)
- added R11: 1meg, R1Meg:RESC2012X65N, F.Cu at (120.7, 116.0)
- added R12: 200k, R100k:RESC1005X40N, F.Cu at (144.8, 77.0)
- added R13: 1meg, R1Meg:RESC2012X65N, F.Cu at (159.0, 80.4)
- added R14: 95.3k, R100k:RESC1005X40N, F.Cu at (158.3, 82.9)
- added R15: 20, R20:RESC1005X35N, F.Cu at (155.2, 94.4)
- added R16: 90k, R806:RESC5025X70N, F.Cu at (144.4, 97.9)
- added R17: 10k, R169:RESC1608X50N, F.Cu at (129.0, 116.4)
- added R18: 0.05, R20:RESC1005X35N, F.Cu at (143.9, 106.7)
- added R5: 80.6k, R806:RESC5025X70N, F.Cu at (151.0, 86.3)
- added R6: 16.9k, R169:RESC1608X50N, F.Cu at (140.4, 106.9)
- added R7: 40.2k, R169:RESC1608X50N, F.Cu at (148.3, 101.3)
- added R8: 90.9k, R806:RESC5025X70N, F.Cu at (149.4, 91.4)
- added R9: 40.2k, R169:RESC1608X50N, F.Cu at (133.0, 116.4)
- added U3: LT3798MPMSETRPBF, LT3798:MSOP-16_MSE, F.Cu at (127.3, 94.4)
- added U4: TPS2546RTER, footprints:TPS2546RTER, F.Cu at (109.5, 107.4)
- C1: footprint Capacitor_SMD:CP_Elec_6.3x9.9 -> Capacitor_THT:CP_Radial_D10.0mm_P7.50mm
- TR1: value TEZ6.0-D-1 -> Wuerth_750343373; footprint Transformer_THT:Transformer_Breve_TEZ-38x45 -> Transformer_THT:Transformer_Wuerth_750343373
- moved U1 44.1 mm to (118.1, 91.9)
- moved J2 33.8 mm to (121.6, 103.7), turned to 0 degrees
- moved U2 33.3 mm to (109.5, 102.8)
- moved R4 33.1 mm to (124.9, 115.8)
- moved C1 32.6 mm to (126.2, 86.0)
- moved R3 22.3 mm to (158.5, 86.3)
- moved D1 20.5 mm to (141.0, 92.5), turned to 0 degrees
- moved R2 19.3 mm to (161.3, 89.5)
- moved TR1 18.1 mm to (93.0, 80.6), turned to 0 degrees
- moved J1 16.9 mm to (139.0, 84.7)
- moved C3 16.1 mm to (156.5, 90.9)
Connections:
- net DM renamed DM1
- net DP renamed DP1
- net Vout renamed Vout1
- D1 pad 3: - -> AC1
- D1 pad 4: + -> AC2
- R2 pad 1: Net-(R2-Pad1) -> Vint
- R2 pad 2: Vint -> Stat2
- TR1 pad 1: AC1 -> Net-(D6-Pad2)
- TR1 pad 10: (no net) -> Net-(TR1-Pad10)
- TR1 pad 2: (no net) -> Net-(TR1-Pad2)
- TR1 pad 4: (no net) -> Net-(D5-Pad1)
- TR1 pad 5: AC2 -> Net-(C1-Pad1)
- TR1 pad 6: (no net) -> dcm
- TR1 pad 7: + -> gnd
- TR1 pad 8: (no net) -> Net-(TR1-Pad8)
- TR1 pad 9: - -> Net-(TR1-Pad9)
- U1 pad 3: Net-(C1-Pad1) -> Net-(C8-Pad1)
- U2 pad 4: Net-(R2-Pad1) -> Stat2
- U2 pad 9: Net-(U2-Pad9) -> Stat1
Routing:
- net Net-(R4-Pad1): track 4.64 -> 0.00 mm
Other:
- board outline removed

Commit message: footprints finalised
Parts:
- removed TR1: Wuerth_750343373, Transformer_THT:Transformer_Wuerth_750343373
- added T1: 760875131, 760875131:760875131, F.Cu at (86.7, 40.8)
- D4, D5, D6: footprint 1N4148WS:SODFL2512X100N -> Diode_SMD:D_1812_4532Metric_Pad1.30x3.40mm_HandSolder
- moved D3 116.6 mm to (43.3, 69.2)
- moved R7 112.0 mm to (51.2, 45.5), turned to 90 degrees
- moved R8 111.8 mm to (43.4, 55.5)
- moved D1 106.8 mm to (44.7, 46.4)
- moved J1 104.6 mm to (44.7, 39.4), turned to 90 degrees
- moved R15 104.3 mm to (53.7, 70.4)
- moved R13 104.1 mm to (61.7, 43.3), turned to 90 degrees
- moved R11 101.8 mm to (42.2, 51.2)
- moved R10 100.3 mm to (44.1, 64.3)
- moved Q1 99.4 mm to (55.4, 56.8)
- moved C7 89.8 mm to (62.9, 56.3)
- moved C1 88.8 mm to (52.5, 36.6)
- moved R16 87.8 mm to (63.6, 63.5)
- moved C5 87.6 mm to (61.7, 70.2)
- moved D5 87.2 mm to (54.2, 65.0)
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
Commit message: routing done
Parts:
- moved R9 56.8 mm to (51.1, 45.7)
- moved R5 23.1 mm to (108.1, 51.6)
- moved R18 14.3 mm to (87.4, 61.1)
- moved R12 11.9 mm to (70.1, 37.8)
- moved R15 10.9 mm to (62.6, 64.1)
- moved D4 9.46 mm to (86.7, 69.5)
- moved R17 8.56 mm to (108.7, 64.9)
- moved C4 7.49 mm to (76.6, 69.6)
- moved R16 7.13 mm to (70.7, 64.0)
- moved R4 7.11 mm to (109.0, 60.6)
- moved C3 7.03 mm to (81.0, 62.6)
- moved R6 6.59 mm to (109.1, 56.0)
- moved U2 5.97 mm to (108.8, 70.6), turned to 90 degrees
- moved C5 5.01 mm to (66.7, 69.5)
- moved D3 3.87 mm to (46.9, 70.7)
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Routing:
- net gnd: track 0.00 -> 300.6 mm
- net Net-(C1-Pad1): track 0.00 -> 139.0 mm
- net Net-(Q1-Pad3): track 0.00 -> 101.2 mm
- net Vint: track 0.00 -> 95.7 mm, vias 0 -> 4
- net en: track 0.00 -> 63.9 mm, vias 0 -> 2
- net Net-(C9-Pad1): track 0.00 -> 61.5 mm, vias 0 -> 1
- net VinL: track 0.00 -> 60.5 mm, vias 0 -> 1
- net Net-(Q1-Pad1): track 0.00 -> 49.2 mm
- net Net-(D5-Pad1): track 0.00 -> 46.1 mm
- net dcm: track 0.00 -> 44.6 mm, vias 0 -> 1
- net Net-(R3-Pad1): track 0.00 -> 42.2 mm, vias 0 -> 2
- net Stat1: track 0.00 -> 41.0 mm, vias 0 -> 3
- net Net-(C4-Pad1): track 0.00 -> 39.5 mm, vias 0 -> 1
- net Stat2: track 0.00 -> 36.4 mm, vias 0 -> 3
- net Net-(D4-Pad1): track 0.00 -> 29.9 mm
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Other:
- board outline added: 94.2 x 44.5 mm
